File: gnss.kicad_sch (KiCad schematic)
At the start: 36 parts, among them J401 GNSS ANT pads, U401 AT6558R-5N32, X401 TCXO 26MHz, X402 32.768kHz

Commit message: Remove the buck-boost: run straight off a 3.6 V max cell
The TPS63001 and its inductor come out and the battery drives the board
directly, so the rail is renamed +3V3 -> +BATT on every sheet: a net called
3V3 that is really the cell is the kind of label someone connects a charger
to.

SW101 used to switch the converter's EN pin, which is why it was never in
series with the load - the C&K JS series is rated 300 mA and this board
peaks past that. With no EN pin it now drives the gate of Q102, a second
DMG3401LSN-7 back to back with the reverse-block Q101. Q101 keeps its source
on the load side so its body diode conducts forward, which is exactly why it
cannot also be the switch; Q102 faces the other way so an open channel
really disconnects.

R102/C102 are re-used as a 10k/1u gate network giving about 9 ms of soft
start, replacing the converter's. Without it the switch would connect ~70 uF
of rail and IC decoupling straight across a cell that may have ohms of
internal resistance. The 10k stays small against the 100k pull-up so the
gate still reaches 91 % of VBATT.

The R103/R104 sense divider moves from VBATT to the switched +BATT, so it
draws nothing with the board off.

Also fixes assemble.ts rewriting cc1200_balloon.kicad_pro from a fixed
template every build, which was silently resetting the net classes, board
design settings and ERC severities KiCad had written. Found while rebuilding
for this change.

Gates: placement 5/5, routing DRC 0, netlist matches sheets/*.json at 378
endpoints / 76 nets, full-hierarchy ERC 0 errors and the 2 known BME688
address-strap warnings. Build output is byte-identical across runs.

The large .kicad_sch diffs are formatting: the committed set had been opened
and saved by KiCad, which expands the compact s-expressions the generator
writes. Nothing but the power sheet and the rail name changed electrically.

Not done: cc1200_balloon.kicad_pcb still carries U101, L101 and C105 and has
no Q102. It needs Update PCB from Schematic.

Co-Au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
Connections:
- net GNSS_RTC_XI: now also C415.1, X402.1
- net GNSS_RTC_XO: now also C416.1, X402.2
- net +3V3 renamed +BATT
Other:
- moved on the sheet: C401, C402, C403, C404, C405, C406, C407, C408, C409, C410, C411, C412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

Commit message: Rewire the GNSS to the real AT6558R-5N32 pinout
The receiver was wired from an invented pinout. Pin names the part does not
have (VANT_IN, VDD_POR, BBLDO_OUT, VDX, AVDD), numbers to match, and
comments citing data sheet sections that do not exist. Not one of the 40
pins was on the right pad.

Every gate in build.sh passed the whole time, because every gate compares
the design to sheets/gnss.json and that file was the thing that was wrong.
ERC, the netlist compare, footprint resolution and the frame fit all agree
happily about a receiver wired to a part that does not exist.

Rebuilt against the data sheet (DS-AT6558-R v1.0):

- Section 3.2.1 supply scheme: +BATT into VDD_IO (7) and DX_IN (21),
  DX_OUT (22) through L403 into VCORE (23), 1 uF on each of the five
  internal LDO outputs, VX_OUT (2) powering the TCXO and its enable.
- Section 7.1 host interface: UART0 is the NMEA port, GPIO0/TXD0 (19) and
  GPIO1/RXD0 (18) through 22R series. 1PPS moves to GPIO13 (35).
- Section 8.1 bias-T values: L401 33 nH choke, C401 100 nF, C402 100 pF DC
  block, L402 6.8 nH series match.
- nRST (17) left floating as section 2.2 requires. RTC crystal loses its
  load caps, which section 9.5 says it must not have.
- All 41 pads accounted for: 24 on nets, 17 explicitly no-connect.

The symbol is redrawn to one rule set: supplies on the top edge and ground
on the bottom, both in pin-number order; signals on the sides in functional
groups separated by a blank slot, pin-number order within each group.

The land pattern is now generated from the section 10.2 package drawing
instead of patched from a stock KiCad file. Patching had left the nine
paste apertures laid out for a 3.6 mm thermal land on the 3.4 mm one: 73%
coverage ending 0.015 mm from its edge. Now 63% on a recentred 3x3 grid.

Gates: placement 5/5, routing DRC 0, netlist matches sheets/*.json at 352
endpoints / 74 nets, full-hierarchy ERC 0 errors and the 2 known BME688
address-strap warnings, bun test 10/10.

BOM.md and digik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
Parts:
- removed C415, C416: 10p, Capacitor_SMD:C_0402_1005Metric, symbol Device:C
- removed C417, C418, C419: 1u, Capacitor_SMD:C_0402_1005Metric, symbol Device:C
- removed C420, C421: 100n, Capacitor_SMD:C_0402_1005Metric, symbol Device:C
- removed C422: 100m, cc1200_balloon:SuperCap_KEMET_FCS_D10.7mm, symbol Device:C_Polarized
- removed R404, R405: 0R, Resistor_SMD:R_0402_1005Metric, symbol Device:R
- C401: value 470p -> 100n
- C402: value 1u -> 100p
- C404, C406: value 100n -> 4u7; footprint Capacitor_SMD:C_0402_1005Metric -> Capacitor_SMD:C_0603_1608Metric
- C405, C412: value 1u -> 100n
- C407, C408, C410: value 100n -> 1u
- C411: value 10u -> 1u; footprint Capacitor_SMD:C_0603_1608Metric -> Capacitor_SMD:C_0402_1005Metric
- C414: value 100p -> 100m; footprint Capacitor_SMD:C_0402_1005Metric -> cc1200_balloon:SuperCap_KEMET_FCS_D10.7mm; symbol Device:C -> Device:C_Polarized; MPN (none) -> FCS0V104ZFTBR24; now not fitted
- L402: value 4n3 -> 6n8
- R402, R403: value 10k -> 22R
- TP401: value GNSS TMS -> GNSS TCK
- TP402: value GNSS TCK -> GNSS TMS
- X401: MPN UCF4031035LK005000-26MDK -> KT2520K26000ACW33T
- X402: MPN FC3215AN 32.768K-C5NN60KC5 -> FC-135 32.768KA-A5
Connections:
- net +BATT: now also C404.1, C405.1, U401.21 (DX_IN), U401.7 (VDD_IO); no longer C407.1, C408.1, C410.1, C413.1, U401.14 (VDD_IO), U401.22 (VDD_POR), U401.27 (DCDC_IN), U401.3 (VANT_IN), X401.4 (VDD)
- net GND: now also C401.2, C414.2, R401.2; no longer C402.2, R403.2
- net GNSS_ANT_BIAS: now also C401.1, U401.10 (ANT_BIAS); no longer C402.1, U401.2 (ANT_BIAS)
- net GNSS_ANT_FEED: now also C402.1; no longer C401.1
- net GNSS_ONOFF: now also U401.30 (ON_OFF); no longer U401.29 (ON_OFF)
- net GNSS_PPS: now also U401.35 (GPIO13/1PPS); no longer U401.21 (GPIO6/1PPS)
- net GNSS_RX: now also R403.2; no longer R402.2
- net GNSS_RXD_RAW: now also R403.1, U401.18 (GPIO1/RXD0); no longer R402.1, U401.20 (GPIO1/RXD1)
- net GNSS_TCK: now also TP401.1, U401.15 (TCK); no longer TP402.1, U401.18 (TCK)
- net GNSS_TEST: now also R401.1, U401.29 (TEST); no longer R403.1, U401.28 (TEST)
- net GNSS_TMS: now also TP402.1, U401.16 (TMS); no longer TP401.1, U401.17 (TMS)
- net GNSS_TX: now also R402.2; no longer R401.2
- net GNSS_TXD_RAW: now also R402.1; no longer R401.1
- net GNSS_VDD12BK: now also C408.1, U401.5 (VDD12BK); no longer C412.1, U401.32 (VDD12_BK)
- net GNSS_VDD_PLL: now also C410.1, U401.38 (VDD_PLL); no longer U401.37 (VDD_PLL)
- net GNSS_VDD_RF: now also C411.1
- net GNSS_XREF: now also U401.3 (XREF), X401.3 (OUT); no longer C414.2, U401.30 (XREF)
- net GNSS_VX: now reaches X401.1 (Tri-State)
- net GNSS_VX: now also C412.1, U401.2 (VX_OUT), X401.4 (VDD)
- net GNSS_VBCKP: now reaches C414.1
- net GNSS_VBCKP: now also C413.1, U401.6 (VDD_BK); no longer X401.3 (OUT)
- net at L402.1: now also C402.2; no longer C401.2
- net GNSS_RTC_O: now reaches U401.11 (RTC_O)
- net GNSS_RTC_O: now also X402.2
- net GNSS_RTC_I: now reaches U401.12 (RTC_I)
- net GNSS_RTC_I: now also X402.1
- net GNSS_RF_IN: now reaches U401.40 (RF_IN)
- net GNSS_RF_IN: now also L402.2
- removed net GNSS_AVDD: C405.1, U401.6 (AVDD)
- net GNSS_DCDC_SW: no longer names the net of U401.26 (NC)
- net GNSS_DCDC_SW: no longer L403.1
- net GNSS_DVDD: no longer names the net of U401.36 (GPIO14)
- net GNSS_LNA_IN renamed GNSS_VDD_ANA
- net GNSS_VDD_ANA: now also C407.1; no longer L402.2
- net GNSS_RTC_XI: no longer names the net of U401.34 (GPIO12)
- net GNSS_RTC_XI: no longer X402.1
- net GNSS_RTC_XO: no longer names the net of U401.33 (GPIO16)
- net GNSS_RTC_XO: no longer X402.2
- net GNSS_V1P2BB renamed GNSS_VDD12BB
- net GNSS_VDD12BB: no longer C406.1, U401.13 (VDD12_BB)
- net GNSS_VBK: no longer names the net of U401.31 (GPIO10/SCL)
- removed net GNSS_VDX: C404.1, C411.1, L403.2, U401.25 (VDD_BBLDO), U401.35 (VDD_PLDO), U401.4 (VDD_RFLDO)
- net NRST renamed GNSS_VCORE
- net GNSS_VCORE: now also C406.1, L403.2
- new net GNSS_DX_SW: L403.1, U401.22 (DX_OUT)
- no-connect marks 11 -> 17
Other:
- moved on the sheet: C401, C402, C403, C404, C405, C406, C407, C408, C409, C410, C411, C412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
