File: power.kicad_sch (KiCad schematic)
At the start: 18 parts, among them J101 BATT pads, Q101 DMG3401LSN-7, Q102 DMG3401LSN-7, SW101 PWR

Commit message: Clean up schematic. Add component groups to PCB.
Parts:
- removed C101, C106: 22u, Capacitor_SMD:C_0805_2012Metric, symbol Device:C
- removed C102: 1u, Capacitor_SMD:C_0402_1005Metric, symbol Device:C
- removed C104: 10u, Capacitor_SMD:C_0603_1608Metric, symbol Device:C
- removed C107: 100n, Capacitor_SMD:C_0402_1005Metric, symbol Device:C
- removed D101: SMF6.5A, Diode_SMD:D_SOD-123F, symbol Device:D_TVS
- removed H101, H102, H103, H104: M2.5, MountingHole:MountingHole_2.7mm_M2.5_ISO7380, symbol Mechanical:MountingHole
- removed J101: BATT pads, cc1200_balloon:SolderPad_Wire_1x02_P3.0mm, symbol Connector_Generic:Conn_01x02
- removed Q101, Q102: DMG3401LSN-7, Package_TO_SOT_SMD:SOT-23, symbol Transistor_FET:Q_PMOS_GSD
- removed R101, R103, R104: 100k, Resistor_SMD:R_0402_1005Metric, symbol Device:R
- removed R102: 10k, Resistor_SMD:R_0402_1005Metric, symbol Device:R
- removed SW101: PWR, Button_Switch_SMD:SW_SPDT_CK_JS102011SAQN, symbol Switch:SW_SPDT
